Commit message: Update the URDF with more details

File: urdf/robko01.urdf (robot description, URDF)
Before this commit: robot robko01, 6 links, 5 joints
Links:
- removed link base
- removed link r
- added link base_link, mass 2.5; collision box size=0.227 0.154 0.030; visual box size=0.227 0.154 0.030
- added link gripper_main, mass 2.5; collision box size=0.019 0.07 0.019; visual box size=0.019 0.07 0.019
- added link grpper_1, mass 2.5; collision box size=0.044 0.006 0.019; visual box size=0.044 0.006 0.019
- added link grpper_2, mass 2.5; collision box size=0.044 0.006 0.019; visual box size=0.044 0.006 0.019
- added link grpper_3, mass 2.5; collision box size=0.044 0.006 0.019; visual box size=0.044 0.006 0.019
- added link grpper_4, mass 2.5; collision box size=0.044 0.006 0.019; visual box size=0.044 0.006 0.019
- added link grpper_5, mass 2.5; collision box size=0.026 0.013 0.013; visual box size=0.026 0.013 0.013
- added link grpper_6, mass 2.5; collision box size=0.026 0.013 0.013; visual box size=0.026 0.013 0.013
- link elbow: geometry collision box size=0.220 0.050 0.050; visual box size=0.220 0.050 0.050
- link p: mass 2.5 -> None; geometry 
- link shoulder: geometry collision box size=0.085 0.044 0.250; visual box size=0.002 0.073 0.250
- link torso: geometry collision box size=0.167 0.088 0.200; visual box size=0.167 0.002 0.200
Joints:
- added joint gripper_2: type revolute, parent gripper_main, child grpper_2, origin xyz=0.0275 -0.028 0.0 rpy=0.0 0.0 0.0, axis 0.0 0.0 1.0, limit lower=-1.5707963705063 upper=1.5707963705063 effort=10 velocity=3, mimic joint=grpper_1 multiplier=1.0 offset=0.0
- added joint gripper_4: type revolute, parent gripper_main, child grpper_4, origin xyz=0.0275 0.028 0.0 rpy=0.0 0.0 0.0, axis 0.0 0.0 1.0, limit lower=-1.5707963705063 upper=1.5707963705063 effort=10 velocity=3, mimic joint=grpper_1 multiplier=-1.0 offset=0.0
- added joint gripper_5: type revolute, parent grpper_2, child grpper_5, origin xyz=0.044 0.0 0.0 rpy=0.0 0.0 0.0, axis 0.0 0.0 1.0, limit lower=-1.5707963705063 upper=1.5707963705063 effort=10 velocity=3, mimic joint=grpper_1 multiplier=-1.0 offset=0.0
- added joint gripper_6: type revolute, parent grpper_4, child grpper_6, origin xyz=0.044 0.0 0.0 rpy=0.0 0.0 0.0, axis 0.0 0.0 1.0, limit lower=-1.5707963705063 upper=1.5707963705063 effort=10 velocity=3, mimic joint=grpper_1 multiplier=1.0 offset=0.0
- added joint grpper_1: type revolute, parent gripper_main, child grpper_1, origin xyz=0.0275 -0.035 0.0 rpy=0.0 0.0 0.0, axis 0.0 0.0 1.0, limit lower=-1.5707963705063 upper=1.5707963705063 effort=10 velocity=3
- added joint grpper_3: type revolute, parent gripper_main, child grpper_3, origin xyz=0.0275 0.035 0.0 rpy=0.0 0.0 0.0, axis 0.0 0.0 1.0, limit lower=-1.5707963705063 upper=1.5707963705063 effort=10 velocity=3, mimic joint=grpper_1 multiplier=-1.0 offset=0.0
- joint base: origin xyz=0.1 0.0 0.1 rpy=0.0 0.0 0.0 -> xyz=0.0 0.0 0.150 rpy=0.0 0.0 0.0; parent base -> base_link
- joint elbow: origin xyz=0.0 0.0 0.4 rpy=0.0 0.0 0.0 -> xyz=0.0 0.0 0.180 rpy=0.0 0.0 0.0
- joint p: origin xyz=0.43 0.0 0.0 rpy=0.0 0.0 0.0 -> xyz=0.175 0.0 0.0 rpy=0.0 0.0 0.0
- joint r: child r -> gripper_main; origin xyz=0.1 0.0 0.0 rpy=0.0 0.0 0.0 -> xyz=0.0 0.0 0.0 rpy=0.0 0.0 0.0
- joint shoulder: origin xyz=-0.03 0.0 0.18 rpy=0.0 0.0 0.0 -> xyz=0.0 0.0 0.050 rpy=0.0 0.0 0.0

Commit message: Update the URDF with more details

File: urdf/robko01.urdf (robot description, URDF)
Before this commit: robot robko01, 12 links, 11 joints
Links:
- removed link grpper_1
- removed link grpper_2
- removed link grpper_3
- removed link grpper_4
- removed link grpper_5
- removed link grpper_6
- added link gripper_1, mass 2.5; collision box size=0.044 0.006 0.019; visual box size=0.044 0.006 0.019
- added link gripper_2, mass 2.5; collision box size=0.044 0.006 0.019; visual box size=0.044 0.006 0.019
- added link gripper_3, mass 2.5; collision box size=0.044 0.006 0.019; visual box size=0.044 0.006 0.019
- added link gripper_4, mass 2.5; collision box size=0.044 0.006 0.019; visual box size=0.044 0.006 0.019
- added link gripper_5, mass 2.5; collision box size=0.026 0.013 0.013; visual box size=0.026 0.013 0.013
- added link gripper_6, mass 2.5; collision box size=0.026 0.013 0.013; visual box size=0.026 0.013 0.013
- link elbow: geometry collision box size=0.220 0.050 0.050; visual box size=0.220 0.050 0.050
- link gripper_main: geometry collision box size=0.019 0.07 0.019; visual box size=0.019 0.07 0.019
- link p: geometry visual cylinder length=0.500 radius=0.001
- link shoulder: geometry collision box size=0.085 0.044 0.250; visual box size=0.002 0.073 0.250
- link torso: geometry collision box size=0.167 0.088 0.200; visual box size=0.167 0.002 0.200
Joints:
- removed joint grpper_1
- removed joint grpper_3
- added joint gripper_1: type revolute, parent gripper_main, child gripper_1, origin xyz=0.0275 -0.035 0.0 rpy=0.0 0.0 0.0, axis 0.0 0.0 1.0, limit lower=-1.5707963705063 upper=1.5707963705063 effort=10 velocity=3
- added joint gripper_3: type revolute, parent gripper_main, child gripper_3, origin xyz=0.0275 0.035 0.0 rpy=0.0 0.0 0.0, axis 0.0 0.0 1.0, limit lower=-1.5707963705063 upper=1.5707963705063 effort=10 velocity=3, mimic joint=gripper_1 multiplier=-1.0 offset=0.0
- joint gripper_2: child grpper_2 -> gripper_2; mimic joint=grpper_1 multiplier=1.0 offset=0.0 -> joint=gripper_1 multiplier=1.0 offset=0.0
- joint gripper_4: child grpper_4 -> gripper_4; mimic joint=grpper_1 multiplier=-1.0 offset=0.0 -> joint=gripper_1 multiplier=-1.0 offset=0.0
- joint gripper_5: child grpper_5 -> gripper_5; mimic joint=grpper_1 multiplier=-1.0 offset=0.0 -> joint=gripper_1 multiplier=-1.0 offset=0.0; parent grpper_2 -> gripper_2
- joint gripper_6: child grpper_6 -> gripper_6; mimic joint=grpper_1 multiplier=1.0 offset=0.0 -> joint=gripper_1 multiplier=1.0 offset=0.0; parent grpper_4 -> gripper_4

Commit message: Trying to make the robot more realistic

File: urdf/robko01.urdf (robot description, URDF)
Before this commit: robot robko01, 12 links, 11 joints
Links:
- link shoulder: geometry collision box size=0.085 0.044 0.250; visual box size=0.002 0.073 0.180
- link torso: geometry collision box size=0.167 0.088 0.200; visual box size=0.065 0.078 0.002
Joints:
- joint base: origin xyz=0.0 0.0 0.150 rpy=0.0 0.0 0.0 -> xyz=0.0 0.0 0.050 rpy=0.0 0.0 0.0
- joint shoulder: origin xyz=0.0 0.0 0.050 rpy=0.0 0.0 0.0 -> xyz=0.0 0.0 0.150 rpy=0.0 0.0 0.0

Commit message: Make the robot more realistic

File: urdf/robko01.urdf (robot description, URDF)
Before this commit: robot robko01, 12 links, 11 joints
Links:
- link elbow: geometry collision box size=0.220 0.050 0.050; visual box size=0.165 0.050 0.002
- link p: geometry visual box size=0.013 0.013 0.016; visual cylinder length=0.016 radius=0.0075
- link shoulder: geometry collision box size=0.085 0.044 0.250; visual box size=0.002 0.073 0.1778
Joints:
- joint elbow: origin xyz=0.0 0.0 0.180 rpy=0.0 0.0 0.0 -> xyz=0.0 0.0 0.1778 rpy=0.0 0.0 0.0
- joint p: origin xyz=0.175 0.0 0.0 rpy=0.0 0.0 0.0 -> xyz=0.1778 0.0 0.0 rpy=0.0 0.0 0.0

Commit message: Add corrections to URDF P joint

File: urdf/robko01.urdf (robot description, URDF)
Before this commit: robot robko01, 12 links, 11 joints
Joints:
- joint p: limit lower=-1.5707963705063 upper=1.0 effort=10 velocity=3 -> lower=-1.5707963705063 upper=1.5707963705063 effort=10 velocity=3

Commit message: Change center cyclinder of the grypper to main gripper link

File: urdf/robko01.urdf (robot description, URDF)
Before this commit: robot robko01, 12 links, 11 joints
Links:
- link gripper_main: geometry collision box size=0.019 0.07 0.019; visual box size=0.019 0.07 0.019
- link p: geometry visual box size=0.013 0.013 0.016; visual cylinder length=0.016 radius=0.0075

Commit message: Add STL test to URDF

File: urdf/robko01.urdf (robot description, URDF)
Before this commit: robot robko01, 12 links, 11 joints
Links:
- link torso: geometry collision box size=0.167 0.088 0.200; visual box size=0.065 0.078 0.002

Commit message: Update URDF limits

File: urdf/robko01.urdf (robot description, URDF)
Before this commit: robot robko01, 12 links, 11 joints
Joints:
- joint gripper_1: limit lower=-1.5707963705063 upper=1.5707963705063 effort=10 velocity=3 -> lower=-0.6 upper=0.6 effort=10 velocity=3

Commit message: Rename links and joints

File: urdf/robko01.urdf (robot description, URDF)
Before this commit: robot robko01, 12 links, 11 joints
Links:
- removed link gripper_1
- removed link gripper_2
- removed link gripper_3
- removed link gripper_4
- removed link gripper_5
- removed link gripper_6
- added link finger_1, mass 2.5; collision box size=0.044 0.006 0.019; visual box size=0.044 0.006 0.019
- added link finger_2, mass 2.5; collision box size=0.044 0.006 0.019; visual box size=0.044 0.006 0.019
- added link finger_3, mass 2.5; collision box size=0.044 0.006 0.019; visual box size=0.044 0.006 0.019
- added link finger_4, mass 2.5; collision box size=0.044 0.006 0.019; visual box size=0.044 0.006 0.019
- added link fingertip_l, mass 2.5; collision box size=0.026 0.013 0.013; visual box size=0.026 0.013 0.013
- added link fingertip_r, mass 2.5; collision box size=0.026 0.013 0.013; visual box size=0.026 0.013 0.013
- link torso: geometry collision box size=0.167 0.088 0.200; visual box size=0.065 0.078 0.002
Joints:
- removed joint gripper_1
- removed joint gripper_2
- removed joint gripper_3
- removed joint gripper_4
- removed joint gripper_5
- removed joint gripper_6
- added joint finger_1: type revolute, parent gripper_main, child finger_1, origin xyz=0.0275 -0.035 0.0 rpy=0.0 0.0 0.0, axis 0.0 0.0 1.0, limit lower=-0.6 upper=0.6 effort=10 velocity=3
- added joint finger_2: type revolute, parent gripper_main, child finger_2, origin xyz=0.0275 -0.028 0.0 rpy=0.0 0.0 0.0, axis 0.0 0.0 1.0, limit lower=-1.5707963705063 upper=1.5707963705063 effort=10 velocity=3, mimic joint=finger_1 multiplier=1.0 offset=0.0
- added joint finger_3: type revolute, parent gripper_main, child finger_3, origin xyz=0.0275 0.035 0.0 rpy=0.0 0.0 0.0, axis 0.0 0.0 1.0, limit lower=-1.5707963705063 upper=1.5707963705063 effort=10 velocity=3, mimic joint=finger_1 multiplier=-1.0 offset=0.0
- added joint finger_4: type revolute, parent gripper_main, child finger_4, origin xyz=0.0275 0.028 0.0 rpy=0.0 0.0 0.0, axis 0.0 0.0 1.0, limit lower=-1.5707963705063 upper=1.5707963705063 effort=10 velocity=3, mimic joint=finger_1 multiplier=-1.0 offset=0.0
- added joint fingertip_l: type revolute, parent finger_4, child fingertip_l, origin xyz=0.044 0.0 0.0 rpy=0.0 0.0 0.0, axis 0.0 0.0 1.0, limit lower=-1.5707963705063 upper=1.5707963705063 effort=10 velocity=3, mimic joint=finger_1 multiplier=1.0 offset=0.0
- added joint fingertip_r: type revolute, parent finger_2, child fingertip_r, origin xyz=0.044 0.0 0.0 rpy=0.0 0.0 0.0, axis 0.0 0.0 1.0, limit lower=-1.5707963705063 upper=1.5707963705063 effort=10 velocity=3, mimic joint=finger_1 multiplier=-1.0 offset=0.0

Commit message: Update the URDF, colors, axis helpers, colisions, model positions, joint compensations

File: urdf/robko01.urdf (robot description, URDF)
Before this commit: robot robko01, 12 links, 11 joints
Links:
- link base_link: mass 2.5 -> None; geometry collision box size=0.227 0.154 0.030; collision cylinder length=0.005 radius=0.045
- link elbow: geometry collision box size=0.165 0.050 0.002; collision box size=0.1778 0.002 0.050
- link finger_1: geometry collision box size=0.044 0.006 0.014; visual box size=0.044 0.006 0.014
- link finger_2: geometry collision box size=0.044 0.006 0.014; visual box size=0.044 0.006 0.014
- link finger_3: geometry collision box size=0.044 0.006 0.014; visual box size=0.044 0.006 0.014
- link finger_4: geometry collision box size=0.044 0.006 0.014; visual box size=0.044 0.006 0.014
- link fingertip_l: geometry collision box size=0.026 0.013 0.019; collision mesh filename=package://robko01_ros2/meshes/finger_prism.STL scale=0.001 0.001 0.001
- link fingertip_r: geometry collision box size=0.026 0.013 0.019; collision mesh filename=package://robko01_ros2/meshes/finger_prism.STL scale=0.001 0.001 0.001
- link gripper_main: geometry collision box size=0.019 0.07 0.019; collision cylinder length=0.016 radius=0.0075
- link shoulder: geometry collision box size=0.002 0.073 0.1778; collision box size=0.085 0.002 0.1778
- link torso: geometry collision box size=0.065 0.078 0.002; collision box size=0.167 0.002 0.135
Joints:
- joint finger_1: limit lower=-0.6 upper=0.6 effort=10 velocity=3 -> lower=-0.6 upper=0.347 effort=10 velocity=3

Commit message: Update the URDF add meshes

File: urdf/robko01.urdf (robot description, URDF)
Before this commit: robot robko01, 12 links, 11 joints
Links:
- link torso: geometry collision box size=0.065 0.078 0.002; collision box size=0.167 0.002 0.135

Commit message: Fix collisions and inertia

File: urdf/robko01.urdf (robot description, URDF)
Before this commit: robot robko01, 12 links, 11 joints
Links:
- link elbow: mass 2.5 -> 10
- link finger_1: mass 2.5 -> 10
- link finger_2: mass 2.5 -> 10
- link finger_3: mass 2.5 -> 10
- link finger_4: mass 2.5 -> 10
- link fingertip_l: mass 2.5 -> 10
- link fingertip_r: mass 2.5 -> 10
- link gripper_main: mass 2.5 -> 10
- link p: mass None -> 10; geometry collision box size=0.013 0.013 0.016; collision cylinder length=0.016 radius=0.0075
- link shoulder: mass 2.5 -> 10
- link torso: mass 2.5 -> 10

Commit message: Comment meshes, due fix the sizes

File: urdf/robko01.urdf (robot description, URDF)
Before this commit: robot robko01, 12 links, 11 joints
Links:
- link fingertip_l: geometry collision box size=0.026 0.013 0.019; visual box size=0.026 0.013 0.019
- link fingertip_r: geometry collision box size=0.026 0.013 0.019; visual box size=0.026 0.013 0.019
