Commit message: Include material definitions

File: description/include.xacro (robot description, xacro)
@@ -2,13 +2,29 @@
 <robot xmlns:xacro="http://www.ros.org/wiki/xacro" >
     <!-- This file is not a robot in and of itself, it just contains some useful tags that could be included in any robot -->
+	<xacro:property name="sheet_thickness" value="0.002" />
     <!-- Specify some colours -->
     <material name="white">
         <color rgba="1 1 1 1"/>
     </material>
+    <material name="black">
+        <color rgba="0.0 0.0 0.0 1.0"/>
+    </material>
+    <material name="dark_gray">
+        <color rgba="0.3 0.3 0.3 1.0"/>
+    </material>
+    <material name="silver">
+        <color rgba="0.7 0.7 0.7 1.0"/>
+    </material>
     <material name="orange">
-        <color rgba="1 0.3 0.1 1"/>
+        <color rgba="0.9 0.6 0.05 1.0"/>
+    </material>
+    <material name="red">
+        <color rgba="1.0 0.2 0.2 1.0"/>
+    </material>
+    <material name="green">
+        <color rgba="0.2 1.0 0.2 1.0"/>
     </material>
     <material name="blue">
-        <color rgba="0.2 0.2 1 1"/>
+        <color rgba="0.2 0.2 1.0 1.0"/>
     </material>
     <!-- Specify some standard inertial calculations https://en.wikipedia.org/wiki/List_of_moments_of_inertia -->
