Commit message: Add Gazebo materials

File: description/gazebo.xacro (robot description, xacro)
@@ -6,4 +6,7 @@
     <!-- Gazebo is unable to use the same <material> tags that are already in the URDF (that RViz uses). -->
     <!-- Instead, we need to add gazebo tags for our links that refer to Gazebo materials -->
+    <gazebo reference="body">
+        <material>Gazebo/Black</material>
+    </gazebo>
     <gazebo reference="base_link">
         <material>Gazebo/Green</material>
