Commit message: Improve robot model

File: description/robko01.urdf.xacro (robot description, xacro)
@@ -18,5 +18,5 @@
 			<inertia ixx="0.001" ixy="0" ixz="0" iyy="0.001" iyz="0" izz="0.001" />
 		</inertial>
-		<collision name="base_link">
+		<collision name="body">
 			<origin  xyz="-0.0685 0.0 0.027" rpy="0.0 0.0 0.0"/>
 			<geometry>
@@ -60,12 +60,10 @@
 			</geometry>
 		</collision>
-		<visual name="base_link">
+		<visual name="body">
 			<origin  xyz="-0.0685 0.0 0.027" rpy="0.0 0.0 0.0"/>
 			<geometry>
 				<box size="0.227 0.154 0.030"/>
 			</geometry>
-			<material name="">
-				<color rgba="0.0 0.0 0.0 1.0"/>
-			</material>
+			<material name="black" />
 		</visual>
 		<visual name="p1">
@@ -74,7 +72,5 @@
 				<cylinder radius="0.045" length="0.005"/>
 			</geometry>
-			<material name="">
-				<color rgba="0.0 0.0 0.0 1.0"/>
-			</material>
+			<material name="black" />
 		</visual>
 		<visual name="ax1">
@@ -83,7 +79,5 @@
 				<cylinder radius="0.010" length="0.085"/>
 			</geometry>
-			<material name="">
-				<color rgba="0.5 0.5 0.5 1.0"/>
-			</material>
+			<material name="blue" />
 		</visual>
 		<visual name="f1">
@@ -92,7 +86,5 @@
 				<cylinder radius="0.010" length="0.0135"/>
 			</geometry>
-			<material name="">
-				<color rgba="0.0 0.0 0.0 1.0"/>
-			</material>
+			<material name="black" />
 		</visual>
 		<visual name="f2">
@@ -101,7 +93,5 @@
 				<cylinder radius="0.010" length="0.0135"/>
 			</geometry>
-			<material name="">
-				<color rgba="0.0 0.0 0.0 1.0"/>
-			</material>
+			<material name="black" />
 		</visual>
 		<visual name="f3">
@@ -110,7 +100,5 @@
 				<cylinder radius="0.010" length="0.0135"/>
 			</geometry>
-			<material name="">
-				<color rgba="0.0 0.0 0.0 1.0"/>
-			</material>
+			<material name="black" />
 		</visual>
 		<visual name="f4">
@@ -119,17 +107,15 @@
 				<cylinder radius="0.010" length="0.0135"/>
 			</geometry>
-			<material name="">
-				<color rgba="0.0 0.0 0.0 1.0"/>
-			</material>
+			<material name="black" />
 		</visual>
 	</link>
 	<joint type="revolute" name="base">
 		<parent link="base_link" />
-		<child link="torso" />
+		<child link="torso_link" />
 		<origin xyz="0.0 0.0 0.050" rpy="0.0 0.0 0.0" />
 		<axis xyz="0.0 0.0 1.0" />
-		<limit upper="1.5707963705063" lower="-1.5707963705063" velocity="3" effort="10" />
-	</joint>
-	<link name="torso">
+		<limit upper="${pi/2}" lower="-${pi/2}" velocity="100" effort="100" />
+	</joint>
+	<link name="torso_link">
 		<inertial>
 			<origin xyz="-0.0385 0.0 0.0" rpy="0.0 0.0 0.0" />
@@ -140,11 +126,11 @@
 			<origin xyz="-0.0385 0.040 0.0675" rpy="0.0 0.0 0.0" />
 			<geometry>
-				<box size="0.167 0.002 0.135"/>
+				<box size="0.167 ${sheet_thickness} 0.135"/>
 			</geometry>
 		</collision>
 		<collision name="torso_6_c">
-			<origin xyz="0.0 0.040 0.150" rpy="1.5707963705063 0.0 0.0" />
-			<geometry>
-				<cylinder radius="0.0425" length="0.002"/>
+			<origin xyz="0.0 0.040 0.150" rpy="${pi/2} 0.0 0.0" />
+			<geometry>
+				<cylinder radius="0.0425" length="${sheet_thickness}"/>
 			</geometry>
 		</collision>
@@ -152,5 +138,5 @@
 			<origin xyz="-0.0385 0.0 0.0" rpy="0.0 0.0 0.0" />
 			<geometry>
-				<box size="0.167 0.078 0.002"/>
+				<box size="0.167 0.078 ${sheet_thickness}"/>
 			</geometry>
 		</collision>
@@ -158,5 +144,5 @@
 			<origin xyz="0.010 0.0 0.060" rpy="0.0 0.0 0.0" />
 			<geometry>
-				<box size="0.065 0.078 0.002"/>
+				<box size="0.065 0.078 ${sheet_thickness}"/>
 			</geometry>
 		</collision>
@@ -164,15 +150,15 @@
 			<origin xyz="-0.0385 -0.040 0.0675" rpy="0.0 0.0 0.0" />
 			<geometry>
-				<box size="0.167 0.002 0.135"/>
+				<box size="0.167 ${sheet_thickness} 0.135"/>
 			</geometry>
 		</collision>
 		<collision name="torso_r_c">
-			<origin xyz="0.0 -0.040 0.150" rpy="1.5707963705063 0.0 0.0" />
-			<geometry>
-				<cylinder radius="0.0425" length="0.002"/>
+			<origin xyz="0.0 -0.040 0.150" rpy="${pi/2} 0.0 0.0" />
+			<geometry>
+				<cylinder radius="0.0425" length="${sheet_thickness}"/>
 			</geometry>
 		</collision>
 		<collision name="m1">
-			<origin xyz="0.0 0.0565 0.090" rpy="1.5707963705063 0.0 0.0" />
+			<origin xyz="0.0 0.0565 0.090" rpy="${pi/2} 0.0 0.0" />
 			<geometry>
 				<cylinder radius="0.03" length="0.025"/>
@@ -180,5 +166,5 @@
 		</collision>
 		<collision name="m2">
-			<origin xyz="-0.095 -0.0565 0.030" rpy="1.5707963705063 0.0 0.0" />
+			<origin xyz="-0.095 -0.0565 0.030" rpy="${pi/2} 0.0 0.0" />
 			<geometry>
 				<cylinder radius="0.03" length="0.025"/>
@@ -186,5 +172,5 @@
 		</collision>
 		<collision name="m3">
-			<origin xyz="-0.095 0.0565 0.030" rpy="1.5707963705063 0.0 0.0" />
+			<origin xyz="-0.095 0.0565 0.030" rpy="${pi/2} 0.0 0.0" />
 			<geometry>
 				<cylinder radius="0.03" length="0.025"/>
@@ -192,5 +178,5 @@
 		</collision>
 		<collision name="m4">
-			<origin xyz="-0.025 -0.0565 0.030" rpy="1.5707963705063 0.0 0.0" />
+			<origin xyz="-0.025 -0.0565 0.030" rpy="${pi/2} 0.0 0.0" />
 			<geometry>
 				<cylinder radius="0.03" length="0.025"/>
@@ -198,5 +184,5 @@
 		</collision>
 		<collision name="m5">
-			<origin xyz="-0.025 0.0565 0.030" rpy="1.5707963705063 0.0 0.0" />
+			<origin xyz="-0.025 0.0565 0.030" rpy="${pi/2} 0.0 0.0" />
 			<geometry>
 				<cylinder radius="0.03" length="0.025"/>
@@ -204,5 +190,5 @@
 		</collision>
 		<collision name="m6">
-			<origin xyz="0.0 -0.0565 0.090" rpy="1.5707963705063 0.0 0.0" />
+			<origin xyz="0.0 -0.0565 0.090" rpy="${pi/2} 0.0 0.0" />
 			<geometry>
 				<cylinder radius="0.03" length="0.025"/>
@@ -214,44 +200,36 @@
 				<cylinder radius="0.001" length="0.500"/>
 			</geometry>
-			<material name="orange"/>
+			<material name="blue"/>
 		</visual>
 		<visual name="torso_l">
 			<origin xyz="-0.0385 0.040 0.0675" rpy="0.0 0.0 0.0" />
 			<geometry>
-				<box size="0.167 0.002 0.135"/>
-			</geometry>
-			<material name="MainColor">
-				<color rgba="0.9 0.6 0.05 1"/>
-			</material>
+				<box size="0.167 ${sheet_thickness} 0.135"/>
+			</geometry>
+			<material name="orange" />
 		</visual>
 		<visual name="torso_vertical_axis">
-			<origin xyz="0.0 0.040 0.150" rpy="1.5707963705063 0.0 0.0" />
-			<geometry>
-				<cylinder radius="0.0425" length="0.002"/>
-			</geometry>
-			<material name="MainColor">
-				<color rgba="0.9 0.6 0.05 1.0"/>
-			</material>
+			<origin xyz="0.0 0.040 0.150" rpy="${pi/2} 0.0 0.0" />
+			<geometry>
+				<cylinder radius="0.0425" length="${sheet_thickness}"/>
+			</geometry>
+			<material name="orange" />
 		</visual>
 		<visual name="torso_c1">
 			<origin xyz="-0.0385 0.0 0.0" rpy="0.0 0.0 0.0" />
 			<geometry>
-				<box size="0.167 0.078 0.002"/>
-			</geometry>
-			<material name="MainColor">
-				<color rgba="0.9 0.6 0.05 1.0"/>
-			</material>
+				<box size="0.167 0.078 ${sheet_thickness}"/>
+			</geometry>
+			<material name="orange" />
 		</visual>
 		<visual name="torso_c2">
 			<origin xyz="0.010 0.0 0.060" rpy="0.0 0.0 0.0" />
 			<geometry>
-				<box size="0.065 0.078 0.002"/>
-			</geometry>
-			<material name="MainColor">
-				<color rgba="0.9 0.6 0.05 1.0"/>
-			</material>
+				<box size="0.065 0.078 ${sheet_thickness}"/>
+			</geometry>
+			<material name="orange" />
 		</visual>
 		<!-- <visual name="torso_c3">
-			<origin xyz="0.20 -0.40 0.0" rpy="0.0 0.0 1.5707963705063" />
+			<origin xyz="0.20 -0.40 0.0" rpy="0.0 0.0 ${pi/2}" />
 			<geometry>
 				<mesh filename="package://robko01_ros2/meshes/base_inside.STL" scale="0.001 0.001 0.001"/>
@@ -262,5 +240,5 @@
 		</visual> -->
 		<visual name="torso_c3">
-			<origin xyz="-0.120 0.037 -0.001" rpy="1.5707963705063 0.0 -1.5707963705063" />
+			<origin xyz="-0.120 0.037 -0.001" rpy="${pi/2} 0.0 -${pi/2}" />
 			<geometry>
 				<mesh filename="package://robko01_ros2/meshes/body_base_bottom.STL" scale="0.001 0.001 0.001"/>
@@ -273,21 +251,17 @@
 			<origin xyz="-0.0385 -0.040 0.0675" rpy="0.0 0.0 0.0" />
 			<geometry>
-				<box size="0.167 0.002 0.135"/>
-			</geometry>
-			<material name="MainColor">
-				<color rgba="0.9 0.6 0.05 1.0"/>
-			</material>
+				<box size="0.167 ${sheet_thickness} 0.135"/>
+			</geometry>
+			<material name="orange" />
 		</visual>
 		<visual name="torso_r_c">
-			<origin xyz="0.0 -0.040 0.150" rpy="1.5707963705063 0.0 0.0" />
-			<geometry>
-				<cylinder radius="0.0425" length="0.002"/>
-			</geometry>
-			<material name="MainColor">
-				<color rgba="0.9 0.6 0.05 1.0"/>
-			</material>
+			<origin xyz="0.0 -0.040 0.150" rpy="${pi/2} 0.0 0.0" />
+			<geometry>
+				<cylinder radius="0.0425" length="${sheet_thickness}"/>
+			</geometry>
+			<material name="orange" />
 		</visual>
 		<!-- <visual name="torso_sides">
-			<origin xyz="-0.120 0.037 -0.001" rpy="1.5707963705063 0.0 -1.5707963705063" />
+			<origin xyz="-0.120 0.037 -0.001" rpy="${pi/2} 0.0 -${pi/2}" />
 			<geometry>
 				<mesh filename="package://robko01_ros2/meshes/base_dynamic.STL" scale="1.001 1.001 1.001"/>
@@ -298,5 +272,26 @@
 		</visual> -->
 		<visual name="m1">
-			<origin xyz="0.0 0.0565 0.090" rpy="1.5707963705063 0.0 0.0" />
+			<origin xyz="0.0 0.0565 0.090" rpy="${pi/2} 0.0 0.0" />
+			<geometry>
+				<cylinder radius="0.03" length="0.025"/>
+			</geometry>
+			<material name="silver" />
+		</visual>
+		<visual name="m2">
+			<origin xyz="-0.095 -0.0565 0.030" rpy="${pi/2} 0.0 0.0" />
+			<geometry>
+				<cylinder radius="0.03" length="0.025"/>
+			</geometry>
+			<material name="silver" />
+		</visual>
+		<visual name="m3">
+			<origin xyz="-0.095 0.0565 0.030" rpy="${pi/2} 0.0 0.0" />
+			<geometry>
+				<cylinder radius="0.03" length="0.025"/>
+			</geometry>
+			<material name="silver" />
+		</visual>
+		<visual name="m4">
+			<origin xyz="-0.025 -0.0565 0.030" rpy="${pi/2} 0.0 0.0" />
 			<geometry>
 				<cylinder radius="0.03" length="0.025"/>
@@ -306,48 +301,17 @@
 			</material>
 		</visual>
-		<visual name="m2">
-			<origin xyz="-0.095 -0.0565 0.030" rpy="1.5707963705063 0.0 0.0" />
-			<geometry>
-				<cylinder radius="0.03" length="0.025"/>
-			</geometry>
-			<material name="MotorGray">
-				<color rgba="0.3 0.3 0.3 1.0"/>
-			</material>
-		</visual>
-		<visual name="m3">
-			<origin xyz="-0.095 0.0565 0.030" rpy="1.5707963705063 0.0 0.0" />
-			<geometry>
-				<cylinder radius="0.03" length="0.025"/>
-			</geometry>
-			<material name="">
-				<color rgba="0.3 0.3 0.3 1.0"/>
-			</material>
-		</visual>
-		<visual name="m4">
-			<origin xyz="-0.025 -0.0565 0.030" rpy="1.5707963705063 0.0 0.0" />
-			<geometry>
-				<cylinder radius="0.03" length="0.025"/>
-			</geometry>
-			<material name="MotorGray">
-				<color rgba="0.3 0.3 0.3 1.0"/>
-			</material>
-		</visual>
 		<visual name="m5">
-			<origin xyz="-0.025 0.0565 0.030" rpy="1.5707963705063 0.0 0.0" />
-			<geometry>
-				<cylinder radius="0.03" length="0.025"/>
-			</geometry>
-			<material name="MotorGray">
-				<color rgba="0.3 0.3 0.3 1.0"/>
-			</material>
+			<origin xyz="-0.025 0.0565 0.030" rpy="${pi/2} 0.0 0.0" />
+			<geometry>
+				<cylinder radius="0.03" length="0.025"/>
+			</geometry>
+			<material name="silver" />
 		</visual>
 		<visual name="m6">
-			<origin xyz="0.0 -0.0565 0.090" rpy="1.5707963705063 0.0 0.0" />
-			<geometry>
-				<cylinder radius="0.03" length="0.025"/>
-			</geometry>
-			<material name="MotorGray">
-				<color rgba="0.3 0.3 0.3 1.0"/>
-			</material>
+			<origin xyz="0.0 -0.0565 0.090" rpy="${pi/2} 0.0 0.0" />
+			<geometry>
+				<cylinder radius="0.03" length="0.025"/>
+			</geometry>
+			<material name="silver" />
 		</visual>
 		<!-- <visual name="base_dynamic">
@@ -371,9 +335,9 @@
 	</link>
 	<joint type="revolute" name="shoulder">
-		<parent link="torso" />
+		<parent link="torso_link" />
 		<child link="shoulder_link" />
 		<origin xyz="0.0 0.0 0.150" rpy="0.0 0.0 0.0"/>
 		<axis xyz="0.0 1.0 0.0" />
-		<limit upper="2.5" lower="-0.8" velocity="3" effort="10" />
+		<limit upper="2.5" lower="-0.8" velocity="100" effort="100" />
 	</joint>
 	<link name="shoulder_link">
@@ -386,11 +350,11 @@
 			<origin xyz="0.0 0.039 0.0889" rpy="0.0 0.0 0.0" />
 			<geometry>
-				<box size="0.085 0.002 0.1778"/>
+				<box size="0.085 ${sheet_thickness} 0.1778"/>
 			</geometry>
 		</collision>
 		<collision name="shoulder_l_c">
-			<origin xyz="0.0 0.039 0.0" rpy="1.5707963705063 0.0 0.0" />
-			<geometry>
-				<cylinder radius="0.0425" length="0.002"/>
+			<origin xyz="0.0 0.039 0.0" rpy="${pi/2} 0.0 0.0" />
+			<geometry>
+				<cylinder radius="0.0425" length="${sheet_thickness}"/>
 			</geometry>
 		</collision>
@@ -398,5 +362,5 @@
 			<origin xyz="-0.0425 0.0025 0.0889" rpy="0.0 0.0 0.0" />
 			<geometry>
-				<box size="0.002 0.073 0.1778"/>
+				<box size="${sheet_thickness} 0.073 0.1778"/>
 			</geometry>
 		</collision>
@@ -404,66 +368,54 @@
 			<origin xyz="0.0 -0.034 0.0889" rpy="0.0 0.0 0.0" />
 			<geometry>
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
Commit message: Swat field names to give names first place in evry tag, this will make it easy to read and comprihande

File: description/robko01.urdf.xacro (robot description, xacro)
@@ -110,5 +110,5 @@
 		</visual>
 	</link>
-	<joint type="revolute" name="base">
+	<joint name="base" type="revolute">
 		<parent link="base_link" />
 		<child link="torso_link" />
@@ -334,5 +334,5 @@
 		</visual> -->
 	</link>
-	<joint type="revolute" name="shoulder">
+	<joint name="shoulder" type="revolute">
 		<parent link="torso_link" />
 		<child link="shoulder_link" />
@@ -420,5 +420,5 @@
 		</visual>
 	</link>
-	<joint type="revolute" name="elbow">
+	<joint name="elbow" type="revolute">
 		<parent link="shoulder_link" />
 		<child link="elbow_link" />
@@ -506,5 +506,5 @@
 		</visual>
 	</link>
-	<joint type="revolute" name="p">
+	<joint name="p" type="revolute">
 		<parent link="elbow_link" />
 		<child link="p_link" />
@@ -568,5 +568,5 @@
 		</visual>
 	</link>
-	<joint type="revolute" name="r">
+	<joint name="r" type="revolute">
 		<parent link="p_link" />
 		<child link="gripper_main" />
@@ -624,5 +624,5 @@
 		</visual>
 	</link>
-	<joint type="revolute" name="finger_1">
+	<joint name="finger_1" type="revolute">
 		<parent link="gripper_main" />
 		<child link="finger_1_link" />
@@ -632,5 +632,5 @@
 		<!-- <limit upper="0.6" lower="-0.6" velocity="100" effort="100" /> -->
 	</joint>
-	<joint type="revolute" name="finger_2">
+	<joint name="finger_2" type="revolute">
 		<parent link="gripper_main" />
 		<child link="finger_2_link" />
@@ -640,5 +640,5 @@
 		<mimic joint="finger_1" multiplier="1.0" offset="0.0" />
 	</joint>
-	<joint type="revolute" name="finger_3">
+	<joint name="finger_3" type="revolute">
 		<parent link="gripper_main" />
 		<child link="finger_3_link" />
@@ -648,5 +648,5 @@
 		<mimic joint="finger_1" multiplier="-1.0" offset="0.0" />
 	</joint>
-	<joint type="revolute" name="finger_4">
+	<joint name="finger_4" type="revolute">
 		<parent link="gripper_main" />
 		<child link="finger_4_link" />
@@ -736,5 +736,5 @@
 		</visual>
 	</link>
-	<joint type="revolute" name="fingertip_r">
+	<joint name="fingertip_r" type="revolute">
 		<parent link="finger_2_link" />
 		<child link="fingertip_r_link" />
