Commit message: STAGE for backup

File: description/robko01.urdf.xacro (robot description, xacro)
@@ -18,92 +18,43 @@
 			<inertia ixx="0.001" ixy="0" ixz="0" iyy="0.001" iyz="0" izz="0.001" />
 		</inertial>
-		<collision name="body">
-			<origin  xyz="-0.0685 0.0 0.027" rpy="0.0 0.0 0.0"/>
-			<geometry>
-				<box size="0.227 0.154 0.030"/>
-			</geometry>
-		</collision>
-		<collision name="p1">
-			<origin xyz="0.0 0.0 0.0425" rpy="0.0 0.0 0.0" />
-			<geometry>
-				<cylinder radius="0.045" length="0.005"/>
-			</geometry>
-		</collision>
-		<collision name="ax1">
-			<origin xyz="0.0 0.0 0.0825" rpy="0.0 0.0 0.0" />
-			<geometry>
-				<cylinder radius="0.010" length="0.085"/>
-			</geometry>
-		</collision>
-		<collision name="f1">
-			<origin xyz="0.0315 0.0635 0.00675" rpy="0.0 0.0 0.0" />
-			<geometry>
-				<cylinder radius="0.010" length="0.0135"/>
-			</geometry>
-		</collision>
-		<collision name="f2">
-			<origin xyz="0.0315 -0.0635 0.00675" rpy="0.0 0.0 0.0" />
-			<geometry>
-				<cylinder radius="0.010" length="0.0135"/>
-			</geometry>
-		</collision>
-		<collision name="f3">
-			<origin xyz="-0.1675 0.0635 0.00675" rpy="0.0 0.0 0.0" />
-			<geometry>
-				<cylinder radius="0.010" length="0.0135"/>
-			</geometry>
-		</collision>
-		<collision name="f4">
-			<origin xyz="-0.1675 -0.0635 0.00675" rpy="0.0 0.0 0.0" />
-			<geometry>
-				<cylinder radius="0.010" length="0.0135"/>
-			</geometry>
-		</collision>
-		<visual name="body">
-			<origin  xyz="-0.0685 0.0 0.027" rpy="0.0 0.0 0.0"/>
-			<geometry>
-				<box size="0.227 0.154 0.030"/>
-			</geometry>
-			<material name="black" />
-		</visual>
-		<visual name="p1">
-			<origin xyz="0.0 0.0 0.0425" rpy="0.0 0.0 0.0" />
-			<geometry>
-				<cylinder radius="0.045" length="0.005"/>
-			</geometry>
-			<material name="black" />
-		</visual>
-		<visual name="ax1">
-			<origin xyz="0.0 0.0 0.0825" rpy="0.0 0.0 0.0" />
-			<geometry>
-				<cylinder radius="0.010" length="0.085"/>
-			</geometry>
-			<material name="blue" />
-		</visual>
 		<visual name="f1">
-			<origin xyz="0.0315 0.0635 0.00675" rpy="0.0 0.0 0.0" />
-			<geometry>
-				<cylinder radius="0.010" length="0.0135"/>
+			<origin xyz="0.0315 0.0635 0.0" rpy="0.0 0.0 0.0" />
+			<geometry>
+				<mesh filename="package://robko01_ros2/meshes/base_foot.STL" scale="0.001 0.001 0.001"/>
 			</geometry>
 			<material name="black" />
 		</visual>
 		<visual name="f2">
-			<origin xyz="0.0315 -0.0635 0.00675" rpy="0.0 0.0 0.0" />
-			<geometry>
-				<cylinder radius="0.010" length="0.0135"/>
+			<origin xyz="0.0315 -0.0635 0.0" rpy="0.0 0.0 0.0" />
+			<geometry>
+				<mesh filename="package://robko01_ros2/meshes/base_foot.STL" scale="0.001 0.001 0.001"/>
 			</geometry>
 			<material name="black" />
 		</visual>
 		<visual name="f3">
-			<origin xyz="-0.1675 0.0635 0.00675" rpy="0.0 0.0 0.0" />
-			<geometry>
-				<cylinder radius="0.010" length="0.0135"/>
+			<origin xyz="-0.1675 0.0635 0.0" rpy="0.0 0.0 0.0" />
+			<geometry>
+				<mesh filename="package://robko01_ros2/meshes/base_foot.STL" scale="0.001 0.001 0.001"/>
 			</geometry>
 			<material name="black" />
 		</visual>
 		<visual name="f4">
-			<origin xyz="-0.1675 -0.0635 0.00675" rpy="0.0 0.0 0.0" />
-			<geometry>
-				<cylinder radius="0.010" length="0.0135"/>
+			<origin xyz="-0.1675 -0.0635 0.0" rpy="0.0 0.0 0.0" />
+			<geometry>
+				<mesh filename="package://robko01_ros2/meshes/base_foot.STL" scale="0.001 0.001 0.001"/>
+			</geometry>
+			<material name="black" />
+		</visual>
+		<visual name="base_case">
+			<origin  xyz="-0.065 0.0 0.011" rpy="0.0 0.0 0.0"/>
+			<geometry>
+				<mesh filename="package://robko01_ros2/meshes/base_case.STL" scale="0.001 0.001 0.001"/>
+			</geometry>
+			<material name="black" />
+		</visual>
+		<visual name="base_lid">
+			<origin  xyz="-0.065 0.0 0.011" rpy="0.0 0.0 0.0"/>
+			<geometry>
+				<mesh filename="package://robko01_ros2/meshes/base_lid.STL" scale="0.001 0.001 0.001"/>
 			</geometry>
 			<material name="black" />
@@ -123,76 +74,4 @@
 			<inertia ixx="0.001" ixy="0" ixz="0" iyy="0.001" iyz="0" izz="0.001" />
 		</inertial>
-		<collision name="torso_l">
-			<origin xyz="-0.0385 0.040 0.0675" rpy="0.0 0.0 0.0" />
-			<geometry>
-				<box size="0.167 ${sheet_thickness} 0.135"/>
-			</geometry>
-		</collision>
-		<collision name="torso_6_c">
-			<origin xyz="0.0 0.040 0.150" rpy="${pi/2} 0.0 0.0" />
-			<geometry>
-				<cylinder radius="0.0425" length="${sheet_thickness}"/>
-			</geometry>
-		</collision>
-		<collision name="torso_c1">
-			<origin xyz="-0.0385 0.0 0.0" rpy="0.0 0.0 0.0" />
-			<geometry>
-				<box size="0.167 0.078 ${sheet_thickness}"/>
-			</geometry>
-		</collision>
-		<collision name="torso_c2">
-			<origin xyz="0.010 0.0 0.060" rpy="0.0 0.0 0.0" />
-			<geometry>
-				<box size="0.065 0.078 ${sheet_thickness}"/>
-			</geometry>
-		</collision>
-		<collision name="torso_r">
-			<origin xyz="-0.0385 -0.040 0.0675" rpy="0.0 0.0 0.0" />
-			<geometry>
-				<box size="0.167 ${sheet_thickness} 0.135"/>
-			</geometry>
-		</collision>
-		<collision name="torso_r_c">
-			<origin xyz="0.0 -0.040 0.150" rpy="${pi/2} 0.0 0.0" />
-			<geometry>
-				<cylinder radius="0.0425" length="${sheet_thickness}"/>
-			</geometry>
-		</collision>
-		<collision name="m1">
-			<origin xyz="0.0 0.0565 0.090" rpy="${pi/2} 0.0 0.0" />
-			<geometry>
-				<cylinder radius="0.03" length="0.025"/>
-			</geometry>
-		</collision>
-		<collision name="m2">
-			<origin xyz="-0.095 -0.0565 0.030" rpy="${pi/2} 0.0 0.0" />
-			<geometry>
-				<cylinder radius="0.03" length="0.025"/>
-			</geometry>
-		</collision>
-		<collision name="m3">
-			<origin xyz="-0.095 0.0565 0.030" rpy="${pi/2} 0.0 0.0" />
-			<geometry>
-				<cylinder radius="0.03" length="0.025"/>
-			</geometry>
-		</collision>
-		<collision name="m4">
-			<origin xyz="-0.025 -0.0565 0.030" rpy="${pi/2} 0.0 0.0" />
-			<geometry>
-				<cylinder radius="0.03" length="0.025"/>
-			</geometry>
-		</collision>
-		<collision name="m5">
-			<origin xyz="-0.025 0.0565 0.030" rpy="${pi/2} 0.0 0.0" />
-			<geometry>
-				<cylinder radius="0.03" length="0.025"/>
-			</geometry>
-		</collision>
-		<collision name="m6">
-			<origin xyz="0.0 -0.0565 0.090" rpy="${pi/2} 0.0 0.0" />
-			<geometry>
-				<cylinder radius="0.03" length="0.025"/>
-			</geometry>
-		</collision>
 		<visual name="torso_axis">
 			<origin xyz="0.0 0.0 0.0" rpy="0.0 0.0 0.0" />
@@ -202,134 +81,41 @@
 			<material name="blue"/>
 		</visual>
-		<visual name="torso_l">
-			<origin xyz="-0.0385 0.040 0.0675" rpy="0.0 0.0 0.0" />
-			<geometry>
-				<box size="0.167 ${sheet_thickness} 0.135"/>
-			</geometry>
-			<material name="orange" />
-		</visual>
-		<visual name="torso_vertical_axis">
-			<origin xyz="0.0 0.040 0.150" rpy="${pi/2} 0.0 0.0" />
-			<geometry>
-				<cylinder radius="0.0425" length="${sheet_thickness}"/>
-			</geometry>
-			<material name="orange" />
-		</visual>
-		<visual name="torso_c1">
-			<origin xyz="-0.0385 0.0 0.0" rpy="0.0 0.0 0.0" />
-			<geometry>
-				<box size="0.167 0.078 ${sheet_thickness}"/>
-			</geometry>
-			<material name="orange" />
-		</visual>
-		<visual name="torso_c2">
-			<origin xyz="0.010 0.0 0.060" rpy="0.0 0.0 0.0" />
-			<geometry>
-				<box size="0.065 0.078 ${sheet_thickness}"/>
-			</geometry>
-			<material name="orange" />
-		</visual>
-		<!-- <visual name="torso_c3">
-			<origin xyz="0.20 -0.40 0.0" rpy="0.0 0.0 ${pi/2}" />
-			<geometry>
-				<mesh filename="package://robko01_ros2/meshes/base_inside.STL" scale="0.001 0.001 0.001"/>
+		<visual name="torso_side_left">
+			<origin xyz="-0.0415 0.0388 0.0925" rpy="-${pi/2} 0.0 0.0" />
+			<geometry>
+				<mesh filename="package://robko01_ros2/meshes/torso_side_left.STL" scale="0.001 0.001 0.001"/>
+			</geometry>
+		</visual>
+		<visual name="torso_bottom">
+			<origin xyz="-0.120 0.037 -0.001" rpy="0.0 0.0 0.0" />
+			<geometry>
+				<mesh filename="package://robko01_ros2/meshes/torso_bottom.STL" scale="0.001 0.001 0.001"/>
 			</geometry>
 			<material name="">
 				<color rgba="0.3 0.5 0.3 1.0"/>
 			</material>
-		</visual> -->
-		<visual name="torso_c3">
-			<origin xyz="-0.120 0.037 -0.001" rpy="${pi/2} 0.0 -${pi/2}" />
-			<geometry>
-				<mesh filename="package://robko01_ros2/meshes/body_base_bottom.STL" scale="0.001 0.001 0.001"/>
-			</geometry>
-			<material name="">
-				<color rgba="0.3 0.5 0.3 1.0"/>
-			</material>
-		</visual>
-		<visual name="torso_r">
-			<origin xyz="-0.0385 -0.040 0.0675" rpy="0.0 0.0 0.0" />
-			<geometry>
-				<box size="0.167 ${sheet_thickness} 0.135"/>
+		</visual>
+		<visual name="torso_side_right">
+			<origin xyz="0.0 -0.0385 0.100" rpy="${pi/2} 0.0 0.0" />
+			<geometry>
+				<mesh filename="package://robko01_ros2/meshes/torso_side_right.STL" scale="0.001 0.001 0.001"/>
 			</geometry>
 			<material name="orange" />
 		</visual>
-		<visual name="torso_r_c">
-			<origin xyz="0.0 -0.040 0.150" rpy="${pi/2} 0.0 0.0" />
-			<geometry>
-				<cylinder radius="0.0425" length="${sheet_thickness}"/>
-			</geometry>
-			<material name="orange" />
-		</visual>
-		<!-- <visual name="torso_sides">
-			<origin xyz="-0.120 0.037 -0.001" rpy="${pi/2} 0.0 -${pi/2}" />
-			<geometry>
-				<mesh filename="package://robko01_ros2/meshes/base_dynamic.STL" scale="1.001 1.001 1.001"/>
-			</geometry>
-			<material name="">
-				<color rgba="0.3 0.5 0.3 1.0"/>
-			</material>
-		</visual> -->
-		<visual name="m1">
-			<origin xyz="0.0 0.0565 0.090" rpy="${pi/2} 0.0 0.0" />
-			<geometry>
-				<cylinder radius="0.03" length="0.025"/>
-			</geometry>
-			<material name="silver" />
-		</visual>
-		<visual name="m2">
-			<origin xyz="-0.095 -0.0565 0.030" rpy="${pi/2} 0.0 0.0" />
-			<geometry>
-				<cylinder radius="0.03" length="0.025"/>
-			</geometry>
-			<material name="silver" />
-		</visual>
-		<visual name="m3">
-			<origin xyz="-0.095 0.0565 0.030" rpy="${pi/2} 0.0 0.0" />
-			<geometry>
-				<cylinder radius="0.03" length="0.025"/>
-			</geometry>
-			<material name="silver" />
-		</visual>
-		<visual name="m4">
-			<origin xyz="-0.025 -0.0565 0.030" rpy="${pi/2} 0.0 0.0" />
-			<geometry>
-				<cylinder radius="0.03" length="0.025"/>
-			</geometry>
-			<material name="MotorGray">
-				<color rgba="0.3 0.3 0.3 1.0"/>
-			</material>
-		</visual>
-		<visual name="m5">
-			<origin xyz="-0.025 0.0565 0.030" rpy="${pi/2} 0.0 0.0" />
-			<geometry>
-				<cylinder radius="0.03" length="0.025"/>
-			</geometry>
-			<material name="silver" />
-		</visual>
-		<visual name="m6">
-			<origin xyz="0.0 -0.0565 0.090" rpy="${pi/2} 0.0 0.0" />
-			<geometry>
-				<cylinder radius="0.03" length="0.025"/>
-			</geometry>
-			<material name="silver" />
-		</visual>
-		<!-- <visual name="base_dynamic">
+		<visual name="axis_06x80">
+			<origin xyz="-0.0 0.0 0.0" rpy="0.0 0.0 0.0" />
+			<geometry>
+				<mesh filename="package://robko01_ros2/meshes/axis_06x80.STL" scale="0.001 0.001 0.001"/>
+			</geometry>
+		</visual>
+		<!-- <visual name="Gear_1M_84T_20PA">
 			<origin xyz="0.0 0.0 0.0" rpy="0.0 0.0 0.0" />
 			<geometry>
-				<mesh filename="package://robko01_ros2/meshes/base_dynamic.STL" scale="1.0 1.0 1.0"/>
+				<mesh filename="package://robko01_ros2/meshes/Gear_1M_84T_20PA.STL" scale="0.001 0.001 0.001"/>
 			</geometry>
 			<material name="">
 				<color rgba="0.3 0.3 0.3 1.0"/>
 			</material>
-		</visual> -->
-		<!-- <visual name="body_base_bottom">
-			<origin xyz="0.0 0.0 0.0" rpy="0.0 0.0 0.0" />
-			<geometry>
-				<mesh filename="package://robko01_ros2/meshes/body_base_bottom.STL" scale="1.0 1.0 1.0"/>
-			</geometry>
-			<material name="">
-				<color rgba="0.3 0.3 0.3 1.0"/>
-			</material>
+			<material name="silver" />
 		</visual> -->
 	</link>
@@ -347,73 +133,20 @@
 			<inertia ixx="0.001" ixy="0" ixz="0" iyy="0.001" iyz="0" izz="0.001" />
 		</inertial>
-		<collision name="shoulder_l">
-			<origin xyz="0.0 0.039 0.0889" rpy="0.0 0.0 0.0" />
-			<geometry>
-				<box size="0.085 ${sheet_thickness} 0.1778"/>
-			</geometry>
-		</collision>
-		<collision name="shoulder_l_c">
-			<origin xyz="0.0 0.039 0.0" rpy="${pi/2} 0.0 0.0" />
-			<geometry>
-				<cylinder radius="0.0425" length="${sheet_thickness}"/>
-			</geometry>
-		</collision>
-		<collision name="shoulder_c">
-			<origin xyz="-0.0425 0.0025 0.0889" rpy="0.0 0.0 0.0" />
-			<geometry>
-				<box size="${sheet_thickness} 0.073 0.1778"/>
-			</geometry>
-		</collision>
-		<collision name="shoulder_r">
-			<origin xyz="0.0 -0.034 0.0889" rpy="0.0 0.0 0.0" />
-			<geometry>
-				<box size="0.085 ${sheet_thickness} 0.1778"/>
-			</geometry>
-		</collision>
-		<collision name="shoulder_r_c">
-			<origin xyz="0.0 -0.034 0.0" rpy="${pi/2} 0.0 0.0" />
-			<geometry>
-				<cylinder radius="0.0425" length="${sheet_thickness}"/>
-			</geometry>
-		</collision>
-		<visual name="shoulder_axis">
-			<origin xyz="0.0 0.0 0.0" rpy="-${pi/2} 0.0 0.0" />
+		<collision name="shoulder_big_part">
+			<origin xyz="0.0 0.0 0.0" rpy="0.0 0.0 0.0" />
+			<geometry>
+				<mesh filename="package://robko01_ros2/meshes/shoulder_big_part.STL" scale="0.001 0.001 0.001"/>
+			</geometry>
+		</collision>
+		<visual name="torso_axis">
+			<origin xyz="0.0 0.0 0.0" rpy="${pi/2} 0.0 0.0" />
 			<geometry>
 				<cylinder radius="0.001" length="0.500"/>
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
Commit message: STAGE Fix some positions, colisions and models

File: description/robko01.urdf.xacro (robot description, xacro)
@@ -206,14 +206,14 @@
 			</geometry>
 		</collision>
-		<collision name="p_r_c">
-			<origin xyz="0.0 -0.0155 0.0" rpy="${pi/2} 0.0 0.0" />
-			<geometry>
-				<cylinder radius="0.0075" length="0.016"/>
-			</geometry>
-		</collision>
-		<collision name="p_l_c">
-			<origin xyz="0.0 0.0155 0.0" rpy="${pi/2} 0.0 0.0" />
-			<geometry>
-				<cylinder radius="0.0075" length="0.016"/>
+		<collision name="ldg">
+			<origin  xyz="0.0 -0.025 0.0" rpy="-${pi/2} 0.0 0.0"/>
+			<geometry>
+				<mesh filename="package://robko01_ros2/meshes/gear_bevel_1.5M20T_20PA_11FW.STL" scale="0.001 0.001 0.001"/>
+			</geometry>
+		</collision>
+		<collision name="rdg">
+			<origin  xyz="0.0 0.025 0.0" rpy="${pi/2} 0.0 0.0"/>
+			<geometry>
+				<mesh filename="package://robko01_ros2/meshes/gear_bevel_1.5M20T_20PA_11FW.STL" scale="0.001 0.001 0.001"/>
 			</geometry>
 		</collision>
@@ -234,17 +234,17 @@
 			<material name="black" />
 		</visual>
-		<visual name="p_r_c">
-			<origin xyz="0.0 -0.0155 0.0" rpy="${pi/2} 0.0 0.0" />
-			<geometry>
-				<cylinder radius="0.0075" length="0.016"/>
-			</geometry>
-			<material name="black" />
-		</visual>
-		<visual name="p_l_c">
-			<origin xyz="0.0 0.0155 0.0" rpy="${pi/2} 0.0 0.0" />
-			<geometry>
-				<cylinder radius="0.0075" length="0.016"/>
-			</geometry>
-			<material name="black" />
+		<visual name="ldg">
+			<origin  xyz="0.0 -0.025 0.0" rpy="-${pi/2} 0.0 0.0"/>
+			<geometry>
+				<mesh filename="package://robko01_ros2/meshes/gear_bevel_1.5M20T_20PA_11FW.STL" scale="0.001 0.001 0.001"/>
+			</geometry>
+			<material name="orange" />
+		</visual>
+		<visual name="rdg">
+			<origin  xyz="0.0 0.025 0.0" rpy="${pi/2} 0.0 0.0"/>
+			<geometry>
+				<mesh filename="package://robko01_ros2/meshes/gear_bevel_1.5M20T_20PA_11FW.STL" scale="0.001 0.001 0.001"/>
+			</geometry>
+			<material name="orange" />
 		</visual>
 	</link>
@@ -262,4 +262,10 @@
 			<inertia ixx="0.001" ixy="0" ixz="0" iyy="0.001" iyz="0" izz="0.001" />
 		</inertial>
+		<collision name="cdg">
+			<origin xyz="0.025 0.0 0.0" rpy="0.0 -${pi/2} 0.0" />
+			<geometry>
+				<mesh filename="package://robko01_ros2/meshes/gear_bevel_1.5M20T_20PA_11FW.STL" scale="0.001 0.001 0.001"/>
+			</geometry>
+		</collision>
 		<collision name="r">
 			<origin xyz="0.0275 0.0 0.0" rpy="0.0 0.0 0.0" />
@@ -268,19 +274,4 @@
 			</geometry>
 		</collision>
-		<collision name="p_c_c">
-			<origin xyz="0.0125 0.0 0.0" rpy="0.0 ${pi/2} 0.0" />
-			<geometry>
-				<cylinder radius="0.0075" length="0.016"/>
-			</geometry>
-		</collision>
-		<!-- <visual name="p_axis">
-			<origin xyz="0.0275 0.00 0.0" rpy="-${pi/2} 0.0 0.0" />
-			<geometry>
-				<cylinder radius="0.001" length="0.500"/>
-			</geometry>
-			<material name="AxisGreen">
-				<color rgba="0.0 1.0 0.0 1.0"/>
-			</material>
-		</visual> -->
 		<visual name="r_axis">
 			<origin xyz="0.0 0.0 0.0" rpy="0.0 -${pi/2} 0.0" />
@@ -290,4 +281,11 @@
 			<material name="red" />
 		</visual>
+		<visual name="cdg">
+			<origin xyz="0.025 0.0 0.0" rpy="0.0 -${pi/2} 0.0" />
+			<geometry>
+				<mesh filename="package://robko01_ros2/meshes/gear_bevel_1.5M20T_20PA_11FW.STL" scale="0.001 0.001 0.001"/>
+			</geometry>
+			<material name="dark_gray" />
+		</visual>
 		<visual name="r">
 			<origin xyz="0.0275 0.0 0.0" rpy="0.0 0.0 0.0" />
@@ -296,11 +294,4 @@
 			</geometry>
 			<material name="black" />
-		</visual>
-		<visual name="p_c_c">
-			<origin xyz="0.0125 0.0 0.0" rpy="0.0 ${pi/2} 0.0" />
-			<geometry>
-				<cylinder radius="0.0075" length="0.016"/>
-			</geometry>
-			<material name="dark_gray" />
 		</visual>
 	</link>
@@ -445,5 +436,5 @@
 		</visual>
 		<collision name="finger_prism_r">
-			<origin xyz="-0.070 0.003 0.194" rpy="-${pi/2} 0.0 0.0" />
+			<origin xyz="0.0 0.003 0.0" rpy="-${pi/2} 0.0 0.0" />
 			<geometry>
 				<mesh filename="package://robko01_ros2/meshes/finger_prism.STL" scale="0.001 0.001 0.001"/>
@@ -451,5 +442,5 @@
 		</collision>
 		<visual name="finger_prism_r">
-			<origin xyz="-0.070 0.003 0.194" rpy="-${pi/2} 0.0 0.0" />
+			<origin xyz="0.0 0.003 0.0" rpy="-${pi/2} 0.0 0.0" />
 			<geometry>
 				<mesh filename="package://robko01_ros2/meshes/finger_prism.STL" scale="0.001 0.001 0.001"/>
@@ -488,5 +479,5 @@
 		</visual>
 		<collision name="finger_prism_l">
-			<origin xyz="-0.070 -0.0030 -0.194" rpy="${pi/2} 0.0 0.0" />
+			<origin xyz="0.0 -0.0030 0.0" rpy="${pi/2} 0.0 0.0" />
 			<geometry>
 				<mesh filename="package://robko01_ros2/meshes/finger_prism.STL" scale="0.001 0.001 0.001"/>
@@ -494,5 +485,5 @@
 		</collision>
 		<visual name="finger_prism_l">
-			<origin xyz="-0.070 -0.0030 -0.194" rpy="${pi/2} 0.0 0.0" />
+			<origin xyz="0.0 -0.0030 0.0" rpy="${pi/2} 0.0 0.0" />
 			<geometry>
 				<mesh filename="package://robko01_ros2/meshes/finger_prism.STL" scale="0.001 0.001 0.001"/>

Commit message: STAGE Fix some positions and models

File: description/robko01.urdf.xacro (robot description, xacro)
@@ -88,5 +88,5 @@
 		</visual>
 		<visual name="torso_bottom">
-			<origin xyz="-0.120 0.037 -0.001" rpy="0.0 0.0 0.0" />
+			<origin xyz="0.0 0.0 0.0" rpy="0.0 0.0 0.0" />
 			<geometry>
 				<mesh filename="package://robko01_ros2/meshes/torso_bottom.STL" scale="0.001 0.001 0.001"/>
@@ -97,5 +97,5 @@
 		</visual>
 		<visual name="torso_side_right">
-			<origin xyz="0.0 -0.0385 0.100" rpy="${pi/2} 0.0 0.0" />
+			<origin xyz="0.0 -0.0 0.0" rpy="${pi/2} 0.0 0.0" />
 			<geometry>
 				<mesh filename="package://robko01_ros2/meshes/torso_side_right.STL" scale="0.001 0.001 0.001"/>

Commit message: Clear positions in xacro

File: description/robko01.urdf.xacro (robot description, xacro)
@@ -82,5 +82,5 @@
 		</visual>
 		<visual name="torso_side_left">
-			<origin xyz="-0.0415 0.0388 0.0925" rpy="-${pi/2} 0.0 0.0" />
+			<origin xyz="0.0 0.0 0.0" rpy="0.0 0.0 0.0" />
 			<geometry>
 				<mesh filename="package://robko01_ros2/meshes/torso_side_left.STL" scale="0.001 0.001 0.001"/>
@@ -97,5 +97,5 @@
 		</visual>
 		<visual name="torso_side_right">
-			<origin xyz="0.0 -0.0 0.0" rpy="${pi/2} 0.0 0.0" />
+			<origin xyz="0.0 0.0 0.0" rpy="0.0 0.0 0.0" />
 			<geometry>
 				<mesh filename="package://robko01_ros2/meshes/torso_side_right.STL" scale="0.001 0.001 0.001"/>
@@ -104,5 +104,5 @@
 		</visual>
 		<visual name="axis_06x80">
-			<origin xyz="-0.0 0.0 0.0" rpy="0.0 0.0 0.0" />
+			<origin xyz="0.0 0.0 0.0" rpy="0.0 0.0 0.0" />
 			<geometry>
 				<mesh filename="package://robko01_ros2/meshes/axis_06x80.STL" scale="0.001 0.001 0.001"/>

Commit message: Cleanup XACRO

File: description/robko01.urdf.xacro (robot description, xacro)
@@ -144,4 +144,5 @@
 				<cylinder radius="0.001" length="0.500"/>
 			</geometry>
+			<material name="green"/>
 		</visual>
 		<visual name="shoulder_big_part">
@@ -167,7 +168,7 @@
 		</inertial>
 		<collision name="elbow_big_part">
-			<origin xyz="0.0889 0.025 0.0" rpy="0.0 0.0 0.0" />
-			<geometry>
-				<box size="0.1778 ${sheet_thickness} 0.050"/>
+			<origin  xyz="0.0 0.0 0.0" rpy="0.0 0.0 0.0"/>
+			<geometry>
+				<mesh filename="package://robko01_ros2/meshes/elbow_big_part.STL" scale="0.001 0.001 0.001"/>
 			</geometry>
 		</collision>
